Commit message: Cleanup meshes and document holistic animation overhaul

File: mobile_manipulator_PPR_base_corrected_sltRdcd.urdf (robot description, URDF)
Before this commit: robot Robot, 12 links, 11 joints
Links:
- link abstract_chassis_link: geometry collision mesh filename=package://meshes/stl_output/base_link_reduced.STL; visual mesh filename=package://meshes/stl_output/base_link_reduced.STL
- link left_arm_base_link: geometry collision mesh filename=package://meshes/stl_output/left_arm_base_link_reduced.STL; visual mesh filename=package://meshes/stl_output/left_arm_base_link_reduced.STL
- link left_arm_link1: geometry collision mesh filename=package://meshes/stl_output/left_arm_link1_reduced.STL; visual mesh filename=package://meshes/stl_output/left_arm_link1_reduced.STL
- link left_arm_link2: geometry collision mesh filename=package://meshes/stl_output/left_arm_link2_reduced.STL; visual mesh filename=package://meshes/stl_output/left_arm_link2_reduced.STL
- link left_arm_link3: geometry collision mesh filename=package://meshes/stl_output/left_arm_link3_reduced.STL; visual mesh filename=package://meshes/stl_output/left_arm_link3_reduced.STL
- link left_arm_link4: geometry collision mesh filename=package://meshes/stl_output/left_arm_link4_reduced.STL; visual mesh filename=package://meshes/stl_output/left_arm_link4_reduced.STL
- link left_arm_link5: geometry collision mesh filename=package://meshes/stl_output/left_arm_link5_reduced.STL; visual mesh filename=package://meshes/stl_output/left_arm_link5_reduced.STL
- link left_arm_link6: geometry collision mesh filename=package://meshes/stl_output/left_arm_link6_reduced.STL; visual mesh filename=package://meshes/stl_output/left_arm_link6_reduced.STL
- link left_gripper_link: geometry collision mesh filename=package://meshes/stl_output/end_effector_reduced.STL; visual mesh filename=package://meshes/stl_output/end_effector_reduced.STL
