Commit message: Align animation and collision pipeline with updated URDF

File: mobile_manipulator_PPR_base_corrected.urdf (robot description, URDF)
Before this commit: robot Robot, 12 links, 11 joints
Links:
- link abstract_chassis_link: mass 1.00000000 -> 50.96231322; geometry collision mesh filename=package://meshes/base_link.STL; visual mesh filename=package://meshes/base_link.STL
- link left_arm_base_link: mass 1.65800000 -> 1.658; geometry collision mesh filename=package://meshes/left_arm_base_link.STL; visual mesh filename=package://meshes/left_arm_base_link.STL
- link left_arm_link1: mass 1.16400000 -> 1.164; geometry collision mesh filename=package://meshes/left_arm_link1.STL; visual mesh filename=package://meshes/left_arm_link1.STL
- link left_arm_link2: mass 1.30000000 -> 1.3; geometry collision mesh filename=package://meshes/left_arm_link2.STL; visual mesh filename=package://meshes/left_arm_link2.STL
- link left_arm_link3: mass 0.81800000 -> 0.818; geometry collision mesh filename=package://meshes/left_arm_link3.STL; visual mesh filename=package://meshes/left_arm_link3.STL
- link left_arm_link4: mass 0.69800000 -> 0.698; geometry collision mesh filename=package://meshes/left_arm_link4.STL; visual mesh filename=package://meshes/left_arm_link4.STL
- link left_arm_link5: mass 0.41700000 -> 0.417; geometry collision mesh filename=package://meshes/left_arm_link5.STL; visual mesh filename=package://meshes/left_arm_link5.STL
- link left_arm_link6: mass 0.03700000 -> 0.037; geometry collision mesh filename=package://meshes/left_arm_link6.STL; visual mesh filename=package://meshes/left_arm_link6.STL
- link left_gripper_link: mass 0.60400000 -> 0.604; geometry collision mesh filename=package://meshes/end_effector.STL; visual mesh filename=package://meshes/end_effector.STL
Joints:
- joint left_arm_joint1: axis 0.00000000 1.00000000 0.00000000 -> 0 1 0; limit lower=-2.87980000 upper=2.87980000 effort=0 velocity=0 -> lower=-2.8798 upper=2.8798 effort=40 velocity=1.6; origin xyz=-0.00111490  0.04460000  0.00000000 rpy=0.00000000 0.00000000 0.00000000 -> xyz=-0.0011149 0.0446 0 rpy=0 0 0
- joint left_arm_joint2: axis 0.00000000  0.00000000 -1.00000000 -> 0 0 -1; limit lower=0.00000000 upper=3.22890000 effort=0 velocity=0 -> lower=0 upper=3.2289 effort=40 velocity=1.6; origin xyz=0.00000000 0.10610000 0.00000000 rpy=0.00000000 0.00000000 0.00000000 -> xyz=0 0.1061 0 rpy=0 0 0
- joint left_arm_joint3: axis 0.00000000  0.00000000 -1.00000000 -> 0 0 -1; limit lower=-3.31610000 upper=0.00000000 effort=0 velocity=0 -> lower=-3.3161 upper=0 effort=27 velocity=4.0; origin xyz=-0.34928000  0.01999800  0.00000000 rpy=0.00000000 0.00000000 0.00000000 -> xyz=-0.34928 0.019998 0 rpy=0 0 0
- joint left_arm_joint4: axis 1.00000000 0.00000000 0.00000000 -> 1 0 0; limit lower=-2.87980000 upper=2.87980000 effort=0 velocity=0 -> lower=-2.8798 upper=2.8798 effort=7 velocity=4.0; origin xyz=0.02735000 0.06976700 0.00000000 rpy=0.00000000 0.00000000 0.00000000 -> xyz=0.02735 0.069767 0 rpy=0 0 0
- joint left_arm_joint5: axis 0.00000000 1.00000000 0.00000000 -> 0 1 0; limit lower=-1.65810000 upper=1.65810000 effort=0 velocity=0 -> lower=-1.6581 upper=1.6581 effort=7 velocity=4.0; origin xyz=0.24630000 -0.00049894  0.00000000 rpy=0.00000000 0.00000000 0.00000000 -> xyz=0.2463 -0.00049894 0 rpy=0 0 0
- joint left_arm_joint6: axis 1.00000000 0.00000000 0.00000000 -> 1 0 0; limit lower=-2.87980000 upper=2.87980000 effort=0 velocity=0 -> lower=-2.8798 upper=2.8798 effort=7 velocity=4.0; origin xyz=0.05824900 0.00050025 0.00000000 rpy=0.00000000 0.00000000 0.00000000 -> xyz=0.058249 0.00050025 0 rpy=0 0 0
- joint left_gripper_joint: axis 100 -> 0 0 0; origin xyz=0.10390000 0.00000000 0.00000000 rpy=0.00000000 0.00000000 0.00000000 -> xyz=0.1039 0 0 rpy=0 0 0

Commit message: Add unified chassis control tools and compare runner

File: mobile_manipulator_PPR_base_corrected.urdf (robot description, URDF)
Before this commit: robot Robot, 12 links, 11 joints
Joints:
- joint arm_mount_joint: axis 100 -> 1 0 0
- joint joint_theta: limit lower=-Inf upper=Inf effort=0 velocity=0 -> lower=-Inf upper=Inf effort=0 velocity=1.6
- joint joint_x: axis 0.00000000 0.00000000 1.00000000 -> 1.00000000 0.00000000 0.00000000

Commit message: Update collision mesh catalog and document changes

File: mobile_manipulator_PPR_base_corrected.urdf (robot description, URDF)
Before this commit: robot Robot, 12 links, 11 joints
Links:
- link abstract_chassis_link: geometry collision mesh filename=package://meshes/base_link.STL; visual mesh filename=package://meshes/base_link.STL
- link left_arm_base_link: geometry collision mesh filename=package://meshes/left_arm_base_link.STL; visual mesh filename=package://meshes/left_arm_base_link.STL
- link left_arm_link1: geometry collision mesh filename=package://meshes/left_arm_link1.STL; visual mesh filename=package://meshes/left_arm_link1.STL
- link left_arm_link2: geometry collision mesh filename=package://meshes/left_arm_link2.STL; visual mesh filename=package://meshes/left_arm_link2.STL
- link left_arm_link3: geometry collision mesh filename=package://meshes/left_arm_link3.STL; visual mesh filename=package://meshes/left_arm_link3.STL
- link left_arm_link4: geometry collision mesh filename=package://meshes/left_arm_link4.STL; visual mesh filename=package://meshes/left_arm_link4.STL
- link left_arm_link5: geometry collision mesh filename=package://meshes/left_arm_link5.STL; visual mesh filename=package://meshes/left_arm_link5.STL
- link left_arm_link6: geometry collision mesh filename=package://meshes/left_arm_link6.STL; visual mesh filename=package://meshes/left_arm_link6.STL
- link left_gripper_link: geometry collision mesh filename=package://meshes/end_effector.STL; visual mesh filename=package://meshes/end_effector.STL
